Commit message: added camera link/joint. changed default world in launch file, as the world must contain the plugin for the camera

File: src/sakeths_first_robot_simulation/description/robot.urdf.xacro (robot description, xacro)
@@ -4,4 +4,4 @@
     <!-- Including all parts of the robot in one xacro file-->
     <xacro:include filename = "robot_body.xacro" />
-    <xacro:include filename = "gazebo_control.xacro" />
+    <xacro:include filename = "gazebo_plugins.xacro" />
 </robot>

File: src/sakeths_first_robot_simulation/description/robot_body.xacro (robot description, xacro)
@@ -123,5 +123,5 @@
         <origin xyz = "0.24 0 0"/>
     </joint>
-    <!-- Added a face/visor with two eyes. -->
+    <!-- Added a face/visor with an eye as a camera. -->
     <link name = "visor">
         <visual>
@@ -142,3 +142,29 @@
         <origin xyz = "${chassis_edge} 0 0.15" rpy = "0 0 ${pi}"/>
     </joint>
+    <!-- Camera Link -->
+    <link name = "camera_link">
+        <visual>
+            <origin xyz = "0.025 0 0" /> <!-- Specifies the originating point for models RELATIVE TO THE LINK-->
+            <geometry>
+                <box size = "0.05 0.05 0.05" />
+            </geometry>
+            <material name = "orange" />
+        </visual>
+        <collision>
+            <origin xyz = "0.025 0 0" /> <!-- Specifies the originating point for models RELATIVE TO THE LINK-->
+            <geometry>
+                <box size = "0.05 0.05 0.05" />
+            </geometry>
+        </collision>
+        <!-- Inertial tag-->
+        <xacro:inertial_box mass="0.1" x="0.05" y="0.05" z="0.05">
+            <origin xyz="0.025 0 0" rpy="0 0 0"/>
+        </xacro:inertial_box>
+    </link>
+    <!-- Camera joint-->
+    <joint name = "camera_joint" type = "fixed">
+        <parent link = "visor" />
+        <child link = "camera_link" />
+        <origin xyz = "0 0 0" rpy = "0 0 ${pi}"/>
+    </joint>
 </robot>
