Commit message: max_velocity of robot can now be changed in CONSTANTS.xacro.

File: src/sakeths_first_robot_simulation/description/CONSTANTS.xacro (robot description, xacro)
@@ -5,3 +5,4 @@
     <xacro:property name = "wheel_radius" value = "0.06" />
     <xacro:property name = "wheel_separation" value = "0.3" />
+    <xacro:property name = "max_velocity" value = "15.0" /> <!-- DO NOT INCREASE. OTHERWISE, THIS WILL MESS UP SIMULATION PHYSICS.-->
 </robot>

File: src/sakeths_first_robot_simulation/description/gazebo_plugins.xacro (robot description, xacro)
@@ -25,5 +25,5 @@
         </plugin>
     </gazebo>
-    <!-- GAZEBO CAMERA REFERENCE. -->
+    <!-- GAZEBO CAMERA REFERENCE/PLUGIN. -->
     <gazebo reference="camera_link">
         <sensor name="camera" type="camera">

File: src/sakeths_first_robot_simulation/description/robot_body.xacro (robot description, xacro)
@@ -72,5 +72,5 @@
         <axis xyz = "0 0 -1" />
         <!-- This considers aspects of a joint like torque (effort) and velocity. It is stored in a URDF and NOT a Gazebo tag. -->
-        <limit effort = "0.05" velocity = "10.0" />
+        <limit effort = "0.05" velocity = "${max_velocity}" />
     </joint>
     <!-- LEFT WHEEL (Link and joint)-->
@@ -98,5 +98,5 @@
         <axis xyz = "0 0 1" />
         <!-- This considers aspects of a joint like torque (effort) and velocity. It is stored in a URDF and NOT a Gazebo tag. -->
-        <limit effort = "0.05" velocity = "10.0" />
+        <limit effort = "0.05" velocity = "${max_velocity}" />
     </joint>
     <!-- CASTER WHEEL (Link and Joint)-->
