Commit message: changed cmd_vel msg type to Twist instead of TwistStamped. fixed issues with rviz2 and gazebo driving/turning being in different directions.

File: src/sakeths_first_robot_simulation/description/robot_body.xacro (robot description, xacro)
@@ -69,5 +69,5 @@
         <parent link = "base_link" />
         <child link = "left_wheel_link" />
-        <origin xyz = "0 -0.15 0" rpy = "-${pi/2} 0 ${pi}"/>
+        <origin xyz = "0 -0.15 0" rpy = "-${pi/2} 0 0"/>
         <axis xyz = "0 0 1" />
         <!-- This considers aspects of a joint like torque (effort) and velocity. It is stored in a URDF and NOT a Gazebo tag. -->
@@ -96,5 +96,5 @@
         <child link = "right_wheel_link" />
         <origin xyz = "0 0.15 0" rpy = "${pi/2} 0 ${pi}"/>
-        <axis xyz = "0 0 -1" />
+        <axis xyz = "0 0 1" />
         <!-- This considers aspects of a joint like torque (effort) and velocity. It is stored in a URDF and NOT a Gazebo tag. -->
         <limit effort = "0.05" velocity = "10.0" />

Commit message: reversed left and right wheel links/joints to maintain consistency (right wheel is the wheel from the back, left wheel is the wheel from the back). fixed issues with teleop aligning with gazebo and rviz2.

File: src/sakeths_first_robot_simulation/description/robot_body.xacro (robot description, xacro)
@@ -48,6 +48,6 @@
         </xacro:inertial_box>
     </link>
-    <!-- LEFT WHEEL (Link and joint)-->
-    <link name = "left_wheel_link">
+    <!-- RIGHT WHEEL (Link and joint)-->
+    <link name = "right_wheel_link">
         <visual>
             <geometry>
@@ -66,14 +66,14 @@
         </xacro:inertial_cylinder>
     </link>
-    <joint name = "left_wheel_joint" type = "continuous"> <!-- Continous joint because the wheel can rotate continously (hence, the name)-->
+    <joint name = "right_wheel_joint" type = "continuous"> <!-- Continous joint because the wheel can rotate continously (hence, the name)-->
         <parent link = "base_link" />
-        <child link = "left_wheel_link" />
-        <origin xyz = "0 -0.15 0" rpy = "-${pi/2} 0 0"/>
-        <axis xyz = "0 0 1" />
+        <child link = "right_wheel_link" />
+        <origin xyz = "0 -0.15 0" rpy = "-${pi/2} 0 ${pi}"/>
+        <axis xyz = "0 0 -1" />
         <!-- This considers aspects of a joint like torque (effort) and velocity. It is stored in a URDF and NOT a Gazebo tag. -->
         <limit effort = "0.05" velocity = "10.0" />
     </joint>
-    <!-- RIGHT WHEEL (Link and joint)-->
-    <link name = "right_wheel_link">
+    <!-- LEFT WHEEL (Link and joint)-->
+    <link name = "left_wheel_link">
         <visual>
             <geometry>
@@ -92,7 +92,7 @@
         </xacro:inertial_cylinder>
     </link>
-    <joint name = "right_wheel_joint" type = "continuous">
+    <joint name = "left_wheel_joint" type = "continuous">
         <parent link = "base_link" />
-        <child link = "right_wheel_link" />
+        <child link = "left_wheel_link" />
         <origin xyz = "0 0.15 0" rpy = "${pi/2} 0 ${pi}"/>
         <axis xyz = "0 0 1" />

Commit message: created separate default world with necessary plugins (differential drive, camera, etc.) for better testing)

File: src/sakeths_first_robot_simulation/description/robot_body.xacro (robot description, xacro)
@@ -145,5 +145,5 @@
     <link name = "camera_link">
         <visual>
-            <origin xyz = "0.025 0 0" /> <!-- Specifies the originating point for models RELATIVE TO THE LINK-->
+            <origin xyz = "0.02 0 0" /> <!-- Specifies the originating point for models RELATIVE TO THE LINK-->
             <geometry>
                 <box size = "0.05 0.05 0.05" />
