Commit message: fixed rgbd camera, so ROS2 nodes can get both RGB and depth images w/ full clarity. NOTE: DO NOT TRUST RVIZ2 FOR DISPLAYING RGB OR DEPTH OUTPUTS -- DEPTH IMAGES DO NOT DISPLAY ON RVIZ2.

File: src/sakeths_first_robot_simulation/description/gazebo_plugins.xacro (robot description, xacro)
@@ -27,5 +27,5 @@
     <!-- GAZEBO CAMERA REFERENCE/PLUGIN. -->
     <gazebo reference="camera_link">
-        <sensor name="camera" type="camera">
+        <sensor name="camera" type="rgbd_camera">
             <pose> 0 0 0 0 0 0 </pose>
             <visualize>true</visualize>
@@ -41,5 +41,5 @@
                 <clip>
                     <near>0.05</near>
-                    <far>8.0</far>
+                    <far>15</far>
                 </clip>
             </camera>

File: src/sakeths_first_robot_simulation/description/robot_body.xacro (robot description, xacro)
@@ -145,5 +145,4 @@
     <link name = "camera_link">
         <visual>
-            <origin xyz = "0.02 0 0" /> <!-- Specifies the originating point for models RELATIVE TO THE LINK-->
             <geometry>
                 <box size = "0.05 0.05 0.05" />
@@ -152,5 +151,4 @@
         </visual>
         <collision>
-            <origin xyz = "0.025 0 0" /> <!-- Specifies the originating point for models RELATIVE TO THE LINK-->
             <geometry>
                 <box size = "0.05 0.05 0.05" />
@@ -159,5 +157,5 @@
         <!-- Inertial tag-->
         <xacro:inertial_box mass="0.1" x="0.05" y="0.05" z="0.05">
-            <origin xyz="0.025 0 0" rpy="0 0 0"/>
+            <origin xyz="0.05 0.05 0.05" rpy="0 0 0"/>
         </xacro:inertial_box>
     </link>
@@ -166,5 +164,5 @@
         <parent link = "visor" />
         <child link = "camera_link" />
-        <origin xyz = "0 0 0" rpy = "0 0 ${pi}"/>
+        <origin xyz = "-0.03 0 0" rpy = "0 0 ${pi}"/>
     </joint>
 </robot>

Commit message: changed 'odom' topic to 'wheel_odom' for clarity. created rtabmap launch file. modified gazebo_plugins and robot_body to add optical camera link to correctly display rtabmap point clouds

File: src/sakeths_first_robot_simulation/description/gazebo_plugins.xacro (robot description, xacro)
@@ -45,5 +45,5 @@
             </camera>
             <topic>camera/image_raw</topic>
-            <gz_frame_id>camera_link</gz_frame_id>
+            <gz_frame_id>camera_link_optical</gz_frame_id>
         </sensor>
     </gazebo>

File: src/sakeths_first_robot_simulation/description/robot_body.xacro (robot description, xacro)
@@ -166,3 +166,11 @@
         <origin xyz = "-0.03 0 0" rpy = "0 0 ${pi}"/>
     </joint>
+    <!-- Camera OPTICAL link and joint (since some ROS2 packages use a different convention) -->
+    <link name = "camera_link_optical">
+    </link>
+    <joint name = "camera_optical_joint" type = "fixed">
+        <parent link = "camera_link" />
+        <child link = "camera_link_optical" />
+        <origin xyz = "0 0 0" rpy = "${-pi/2} 0 ${-pi/2}"/>
+    </joint>
 </robot>
